File: qcard-dumper-pcb/QCard.kicad_sch (KiCad schematic)
At the start: 2 parts, among them J1 Conn_02x18_Top_Bottom, U1 AT27C040-70PU

Commit message: Dumper v1
Parts:
- J1: value Conn_02x18_Top_Bottom -> Conn_02x18_Odd_Even; footprint Connector_PinSocket_2.54mm:PinSocket_2x18_P2.54mm_Vertical -> (none); symbol Connector_Generic:Conn_02x18_Top_Bottom -> Connector_Generic:Conn_02x18_Odd_Even
Connections:
- net A0: now also J1.26 (Pin_26); no longer J1.13 (Pin_13)
- net A1: now also J1.24 (Pin_24); no longer J1.12 (Pin_12)
- net A10: now also J1.19 (Pin_19); no longer J1.27 (Pin_27)
- net A11: now also J1.15 (Pin_15)
- net A12: now also J1.10 (Pin_10); no longer J1.5 (Pin_5)
- net A13: now also J1.9 (Pin_9); no longer J1.23 (Pin_23)
- net A14: now also J1.7 (Pin_7); no longer J1.22 (Pin_22)
- net A15: now also J1.8 (Pin_8); no longer J1.4 (Pin_4)
- net A16: now also J1.6 (Pin_6); no longer J1.3 (Pin_3)
- net A17: now also J1.5 (Pin_5); no longer J1.21 (Pin_21)
- net A18: now also J1.3 (Pin_3); no longer J1.20 (Pin_20)
- net A2: now also J1.22 (Pin_22); no longer J1.11 (Pin_11)
- net A3: now also J1.20 (Pin_20); no longer J1.10 (Pin_10)
- net A4: now also J1.18 (Pin_18); no longer J1.9 (Pin_9)
- net A5: now also J1.16 (Pin_16); no longer J1.8 (Pin_8)
- net A6: now also J1.14 (Pin_14); no longer J1.7 (Pin_7)
- net A7: now also J1.12 (Pin_12); no longer J1.6 (Pin_6)
- net A8: now also J1.11 (Pin_11); no longer J1.24 (Pin_24)
- net A9: now also J1.13 (Pin_13); no longer J1.25 (Pin_25)
- net CE: now also J1.21 (Pin_21); no longer J1.28 (Pin_28)
- net D0: now also J1.28 (Pin_28); no longer J1.14 (Pin_14)
- net D1: now also J1.30 (Pin_30); no longer J1.15 (Pin_15)
- net D2: now also J1.32 (Pin_32); no longer J1.16 (Pin_16), J1.34 (Pin_34)
- net D3: now also J1.31 (Pin_31); no longer J1.33 (Pin_33)
- net D4: now also J1.29 (Pin_29); no longer J1.32 (Pin_32)
- net D5: now also J1.27 (Pin_27); no longer J1.31 (Pin_31)
- net D6: now also J1.25 (Pin_25); no longer J1.30 (Pin_30)
- net D7: now also J1.23 (Pin_23); no longer J1.29 (Pin_29)
- net GND: now also J1.33 (Pin_33), J1.34 (Pin_34), J1.4 (Pin_4); no longer J1.1 (Pin_1), J1.17 (Pin_17), J1.36 (Pin_36)
- net OE: now also J1.17 (Pin_17); no longer J1.26 (Pin_26)
- net VCC: now also J1.1 (Pin_1); no longer J1.19 (Pin_19)
Changed lines of the file:
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@@
 (kicad_sch (version 20211123) (generator eeschema)
   (paper "A4")
+  (no_connect (at 165.1 129.54))
   (no_connect (at 139.7 147.32))
-  (no_connect (at 152.4 129.54))
-  (label "CE" (at 165.1 109.22 0)
+  (label "A3" (at 165.1 109.22 0)
     (effects (font (size 1.27 1.27)) (justify left bottom))
   )
@@
     (effects (font (size 1.27 1.27)) (justify left bottom))
   )
-  (label "A17" (at 165.1 91.44 0)
-    (effects (font (size 1.27 1.27)) (justify left bottom))
-  )
-  (label "A15" (at 152.4 93.98 180)
+  (label "A16" (at 165.1 91.44 0)
+    (effects (font (size 1.27 1.27)) (justify left bottom))
+  )
+  (label "A14" (at 152.4 93.98 180)
     (effects (font (size 1.27 1.27)) (justify right bottom))
   )
@@
     (effects (font (size 1.27 1.27)) (justify left bottom))
   )
-  (label "A13" (at 165.1 96.52 0)
+  (label "A12" (at 165.1 96.52 0)
     (effects (font (size 1.27 1.27)) (justify left bottom))
   )
@@
     (effects (font (size 1.27 1.27)) (justify left bottom))
   )
-  (label "D3" (at 165.1 121.92 0)
-    (effects (font (size 1.27 1.27)) (justify left bottom))
-  )
-  (label "A7" (at 152.4 99.06 180)
-    (effects (font (size 1.27 1.27)) (justify right bottom))
-  )
-  (label "D4" (at 165.1 119.38 0)
-    (effects (font (size 1.27 1.27)) (justify left bottom))
-  )
-  (label "D6" (at 165.1 114.3 0)
+  (label "D1" (at 165.1 121.92 0)
+    (effects (font (size 1.27 1.27)) (justify left bottom))
+  )
+  (label "A8" (at 152.4 99.06 180)
+    (effects (font (size 1.27 1.27)) (justify right bottom))
+  )
+  (label "D0" (at 165.1 119.38 0)
+    (effects (font (size 1.27 1.27)) (justify left bottom))
+  )
+  (label "A1" (at 165.1 114.3 0)
     (effects (font (size 1.27 1.27)) (justify left bottom))
   )
@@
     (effects (font (size 1.27 1.27)) (justify left bottom))
   )
-  (label "A10" (at 165.1 106.68 0)
-    (effects (font (size 1.27 1.27)) (justify left bottom))
-  )
-  (label "D7" (at 165.1 111.76 0)
-    (effects (font (size 1.27 1.27)) (justify left bottom))
-  )
-  (label "A14" (at 165.1 93.98 0)
+  (label "A4" (at 165.1 106.68 0)
+    (effects (font (size 1.27 1.27)) (justify left bottom))
+  )
+  (label "A2" (at 165.1 111.76 0)
+    (effects (font (size 1.27 1.27)) (justify left bottom))
+  )
+  (label "A15" (at 165.1 93.98 0)
     (effects (font (size 1.27 1.27)) (justify left bottom))
   )
@@
     (effects (font (size 1.27 1.27)) (justify left bottom))
   )
-  (label "A2" (at 152.4 111.76 180)
+  (label "CE" (at 152.4 111.76 180)
     (effects (font (size 1.27 1.27)) (justify right bottom))
   )
@@
     (effects (font (size 1.27 1.27)) (justify left bottom))
   )
-  (label "A8" (at 165.1 99.06 0)
+  (label "GND" (at 152.4 129.54 180)
+    (effects (font (size 1.27 1.27)) (justify right bottom))
+  )
+  (label "A7" (at 165.1 99.06 0)
     (effects (font (size 1.27 1.27)) (justify left bottom))
   )
@@
     (effects (font (size 1.27 1.27)) (justify left bottom))
   )
-  (label "A18" (at 165.1 88.9 0)
-    (effects (font (size 1.27 1.27)) (justify left bottom))
-  )
-  (label "VCC" (at 165.1 86.36 0)
+  (label "GND" (at 165.1 88.9 0)
+    (effects (font (size 1.27 1.27)) (justify left bottom))
+  )
+  (label "GND" (at 165.1 86.36 0)
     (effects (font (size 1.27 1.27)) (justify left bottom))
   )
@@
     (effects (font (size 1.27 1.27)) (justify left bottom))
   )
-  (label "GND" (at 152.4 88.9 180)
-    (effects (font (size 1.27 1.27)) (justify right bottom))
-  )
-  (label "D5" (at 165.1 116.84 0)
+  (label "A18" (at 152.4 88.9 180)
+    (effects (font (size 1.27 1.27)) (justify right bottom))
+  )
+  (label "A0" (at 165.1 116.84 0)
     (effects (font (size 1.27 1.27)) (justify left bottom))
   )
@@
     (effects (font (size 1.27 1.27)) (justify right bottom))
   )
-  (label "A0" (at 152.4 116.84 180)
+  (label "D6" (at 152.4 116.84 180)
     (effects (font (size 1.27 1.27)) (justify right bottom))
   )
@@
     (effects (font (size 1.27 1.27)) (justify left bottom))
   )
-  (label "GND" (at 152.4 86.36 180)
+  (label "VCC" (at 152.4 86.36 180)
     (effects (font (size 1.27 1.27)) (justify right bottom))
   )
@@
     (effects (font (size 1.27 1.27)) (justify right bottom))
   )
-  (label "A5" (at 152.4 104.14 180)
-    (effects (font (size 1.27 1.27)) (justify right bottom))
-  )
-  (label "D0" (at 152.4 119.38 180)
-    (effects (font (size 1.27 1.27)) (justify right bottom))
-  )
-  (label "A1" (at 152.4 114.3 180)
-    (effects (font (size 1.27 1.27)) (justify right bottom))
-  )
-  (label "A16" (at 152.4 91.44 180)
-    (effects (font (size 1.27 1.27)) (justify right bottom))
-  )
-  (label "A4" (at 152.4 106.68 180)
-    (effects (font (size 1.27 1.27)) (justify right bottom))
-  )
-  (label "GND" (at 165.1 129.54 0)
-    (effects (font (size 1.27 1.27)) (justify left bottom))
-  )
-  (label "D2" (at 152.4 124.46 180)
+  (label "A11" (at 152.4 104.14 180)
+    (effects (font (size 1.27 1.27)) (justify right bottom))
+  )
+  (label "D5" (at 152.4 119.38 180)
+    (effects (font (size 1.27 1.27)) (justify right bottom))
+  )
+  (label "D7" (at 152.4 114.3 180)
+    (effects (font (size 1.27 1.27)) (justify right bottom))
+  )
+  (label "A17" (at 152.4 91.44 180)
+    (effects (font (size 1.27 1.27)) (justify right bottom))
+  )
+  (label "OE" (at 152.4 106.68 180)
+    (effects (font (size 1.27 1.27)) (justify right bottom))
+  )
+  (label "D3" (at 152.4 124.46 180)
     (effects (font (size 1.27 1.27)) (justify right bottom))
   )
@@
     (effects (font (size 1.27 1.27)) (justify left bottom))
   )
-  (label "D1" (at 152.4 121.92 180)
+  (label "D4" (at 152.4 121.92 180)
     (effects (font (size 1.27 1.27)) (justify right bottom))
   )
@@
     (effects (font (size 1.27 1.27)) (justify right bottom))
   )
-  (label "A9" (at 165.1 101.6 0)
+  (label "A6" (at 165.1 101.6 0)
     (effects (font (size 1.27 1.27)) (justify left bottom))
   )
@@
     (effects (font (size 1.27 1.27)) (justify left bottom))
   )
-  (label "A6" (at 152.4 101.6 180)
-    (effects (font (size 1.27 1.27)) (justify right bottom))
-  )
-  (label "A3" (at 152.4 109.22 180)
+  (label "A9" (at 152.4 101.6 180)
+    (effects (font (size 1.27 1.27)) (justify right bottom))
+  )
+  (label "A10" (at 152.4 109.22 180)
     (effects (font (size 1.27 1.27)) (justify right bottom))
   )
@@
     (effects (font (size 1.27 1.27)) (justify left bottom))
   )
-  (label "A12" (at 152.4 96.52 180)
+  (label "A13" (at 152.4 96.52 180)
     (effects (font (size 1.27 1.27)) (justify right bottom))
   )
@@
     (effects (font (size 1.27 1.27)) (justify left bottom))
   )
-  (label "OE" (at 165.1 104.14 0)
+  (label "A5" (at 165.1 104.14 0)
     (effects (font (size 1.27 1.27)) (justify left bottom))
   )
@@
     (pin "9")
   )
-  (symbol (lib_id "Connector_Generic:Conn_02x18_Top_Bottom") (at 157.48 106.68 0) (unit 1)
+  (symbol (lib_id "Connector_Generic:Conn_02x18_Odd_Even") (at 157.48 106.68 0) (unit 1)
     (in_bom yes) (on_board yes) (fields_autoplaced)
-    (property "Reference" "J1" (id 0) (at 158.75 80.01 0))
-    (property "Value" "Conn_02x18_Top_Bottom" (id 1) (at 158.75 82.55 0))
-    (property "Footprint" "Connector_PinSocket_2.54mm:PinSocket_2x18_P2.54mm_Vertical" (id 2) (at 157.48 106.68 0)
+    (property "Reference" "J1" (id 0) (at 158.75 83.82 0))
+    (property "Value" "Conn_02x18_Odd_Even" (id 1) (at 158.75 132.08 0))
+    (property "Footprint" "" (id 2) (at 157.48 106.68 0)
       (effects (font (size 1.27 1.27)) hide)
     )
@@
   (symbol_instances
     (path "/d6be5c00-9669-4734-8400-11015d756ee9"
-      (reference "J1") (unit 1) (value "Conn_02x18_Top_Bottom") (footprint "Connector_PinSocket_2.54mm:PinSocket_2x18_P2.54mm_Vertical")
+      (reference "J1") (unit 1) (value "Conn_02x18_Odd_Even") (footprint "Connector_PinSocket_2.54mm:PinSocket_2x18_P2.54mm_Vertical")
     )
     (path "/97038ab0-55e2-4758-aa99-dc40862dbdca"
