File: qcard-tsop32/QCard.kicad_pcb (KiCad board)
At the start: 2 copper layers, 55 x 45 mm, 6 parts, among them J1 Conn_02x18_Top_Bottom, U1 SST39SF040

Commit message: Better labeling
Parts:
- moved REF** 12.5 mm to (54.5, 67.5)
- moved REF** 12.5 mm to (100.5, 67.5)
- moved JP1 4.40 mm to (62.5, 67.5)
Routing:
- net Net-(J1-Pad18): track 61.7 -> 56.3 mm
- net /PGM: track 14.4 -> 10.1 mm
- net /VCC: track 38.2 -> 35.4 mm
- net /GND: vias 2 -> 3
Other:
- board size 55 x 45 mm -> 55 x 32 mm
- board text added: "1"
- board text added: "18"
- board text added: "19"
- board text added: "36"
- board text added: "PROGRAM / PIN 18"
- board text added: "READ / VIH"
- board text added: "WE#"
- board text removed: "PROGRAM"
- board text removed: "READ"
Changed lines of the file:
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@@
   (net 33 "Net-(J1-Pad18)")
   (footprint "Jumper:SolderJumper-3_P1.3mm_Open_Pad1.0x1.5mm" (layer "F.Cu")
-    (at 58.1 67.4 90)
+    (at 62.5 67.5 90)
     (descr "SMD Solder 3-pad Jumper, 1x1.5mm Pads, 0.3mm gap, open")
     (tags "solder jumper open")
@@
   )
   (footprint "MountingHole:MountingHole_6.4mm_M6" (layer "F.Cu")
-    (at 54.5 55)
+    (at 54.5 67.5)
     (descr "Mounting Hole 6.4mm, no annular, M6")
     (tags "mounting hole 6.4mm no annular m6")
     (attr exclude_from_pos_files exclude_from_bom)
-    (fp_text reference "REF**" (at 0 -7.4) (layer "F.SilkS")
+    (fp_text reference "REF**" (at 0 -7.4) (layer "F.SilkS") hide
       (effects (font (size 1 1) (thickness 0.15)))
     )
@@
     (property "Sheetname" "")
     (attr through_hole)
-    (fp_text reference "U1" (at 0 -5.4525) (layer "F.SilkS")
+    (fp_text reference "U1" (at 0 -5.4525) (layer "F.Fab")
       (effects (font (size 1 1) (thickness 0.15)))
     )
@@
   )
   (footprint "MountingHole:MountingHole_6.4mm_M6" (layer "F.Cu")
-    (at 100.5 55)
+    (at 100.5 67.5)
     (descr "Mounting Hole 6.4mm, no annular, M6")
     (tags "mounting hole 6.4mm no annular m6")
     (attr exclude_from_pos_files exclude_from_bom)
-    (fp_text reference "REF**" (at 0 -7.4) (layer "F.SilkS")
+    (fp_text reference "REF**" (at 0 -7.4) (layer "F.SilkS") hide
       (effects (font (size 1 1) (thickness 0.15)))
     )
@@
     )
   )
-  (gr_line (start 105 84.25) (end 105 50) (layer "Edge.Cuts") (width 0.1))
-  (gr_line (start 50 50) (end 50 84.25) (layer "Edge.Cuts") (width 0.1))
+  (gr_line (start 105 84.25) (end 105 63) (layer "Edge.Cuts") (width 0.1))
+  (gr_line (start 50 63) (end 50 84.25) (layer "Edge.Cuts") (width 0.1))
   (gr_arc (start 54.5 95) (mid 53.792893 94.707107) (end 53.5 94) (layer "Edge.Cuts") (width 0.1))
   (gr_arc (start 101.5 94) (mid 101.207107 94.707107) (end 100.5 95) (layer "Edge.Cuts") (width 0.1))
@@
   (gr_line (start 100.5 95) (end 54.5 95) (layer "Edge.Cuts") (width 0.1))
   (gr_line (start 50 84.25) (end 53.5 84.25) (layer "Edge.Cuts") (width 0.1))
-  (gr_line (start 50 50) (end 105 50) (layer "Edge.Cuts") (width 0.1))
+  (gr_line (start 50 63) (end 105 63) (layer "Edge.Cuts") (width 0.1))
   (gr_line (start 53.5 84.25) (end 53.5 94) (layer "Edge.Cuts") (width 0.1))
   (gr_line (start 101.5 94) (end 101.5 84.25) (layer "Edge.Cuts") (width 0.1))
   (gr_line (start 77.5 50) (end 77.5 95) (layer "User.1") (width 0.15))
-  (gr_text "READ" (at 58.1 70.2) (layer "F.SilkS")
+  (gr_text "36" (at 99 83) (layer "B.SilkS")
+    (effects (font (size 0.5 0.5) (thickness 0.1)) (justify mirror))
+  )
+  (gr_text "19" (at 56 83) (layer "B.SilkS")
+    (effects (font (size 0.5 0.5) (thickness 0.1)) (justify mirror))
+  )
+  (gr_text "READ / VIH" (at 62.5 70.2) (layer "F.SilkS")
     (effects (font (size 0.5 0.5) (thickness 0.1)))
   )
-  (gr_text "PROGRAM" (at 58.1 64.7) (layer "F.SilkS")
+  (gr_text "PROGRAM / PIN 18" (at 62.5 64.75) (layer "F.SilkS")
     (effects (font (size 0.5 0.5) (thickness 0.1)))
   )
-  (gr_text "Q-Chord song cartridge 4Mbit\n${COMPANY} ${ISSUE_DATE}" (at 77.5 54.9) (layer "F.SilkS")
+  (gr_text "Q-Chord song cartridge 4Mbit\n${COMPANY} ${ISSUE_DATE}" (at 77.5 79.5) (layer "F.SilkS")
     (effects (font (size 1.25 1.25) (thickness 0.15)))
   )
+  (gr_text "WE#" (at 64 67.5) (layer "F.SilkS")
+    (effects (font (size 0.5 0.5) (thickness 0.1)) (justify left))
+  )
+  (gr_text "1" (at 56 83) (layer "F.SilkS")
+    (effects (font (size 0.5 0.5) (thickness 0.1)))
+  )
+  (gr_text "18" (at 99 83) (layer "F.SilkS")
+    (effects (font (size 0.5 0.5) (thickness 0.1)))
+  )
+  (segment (start 62.5 68.8) (end 62.5975 68.7025) (width 0.3) (layer "F.Cu") (net 1))
+  (segment (start 62.5975 68.7025) (end 72.201377 68.7025) (width 0.3) (layer "F.Cu") (net 1))
+  (segment (start 58.2 73.1) (end 62.5 68.8) (width 0.3) (layer "F.Cu") (net 1))
+  (segment (start 58.25 76.15) (end 58.3 76.2) (width 0.3) (layer "F.Cu") (net 1))
+  (segment (start 58.2 73.45) (end 58.2 73.1) (width 0.3) (layer "F.Cu") (net 1))
   (segment (start 58.25 73.5) (end 58.2 73.45) (width 0.3) (layer "F.Cu") (net 1))
-  (segment (start 58.25 76.15) (end 58.3 76.2) (width 0.3) (layer "F.Cu") (net 1))
-  (segment (start 58.2 73.45) (end 58.2 68.8) (width 0.3) (layer "F.Cu") (net 1))
-  (segment (start 58.1 68.7) (end 58.1025 68.7025) (width 0.3) (layer "F.Cu") (net 1))
-  (segment (start 58.1025 68.7025) (end 72.201377 68.7025) (width 0.3) (layer "F.Cu") (net 1))
-  (segment (start 58.2 68.8) (end 58.1 68.7) (width 0.3) (layer "F.Cu") (net 1))
   (segment (start 58.25 73.5) (end 58.25 76.15) (width 0.3) (layer "F.Cu") (net 1))
   (via (at 58.25 73.5) (size 0.9) (drill 0.4) (layers "F.Cu" "B.Cu") (net 1))
@@
   (via (at 90 69.75) (size 0.9) (drill 0.4) (layers "F.Cu" "B.Cu") (net 2))
   (via (at 56.3 73.5) (size 0.8) (drill 0.4) (layers "F.Cu" "B.Cu") (free) (net 2))
+  (via (at 100.5 73.5) (size 0.8) (drill 0.4) (layers "F.Cu" "B.Cu") (free) (net 2))
   (segment (start 60.99 89) (end 60.99 78.01) (width 0.25) (layer "F.Cu") (net 3))
   (segment (start 69.297499 69.702501) (end 72.201377 69.702501) (width 0.25) (layer "F.Cu") (net 3))
@@
   (segment (start 94.01 89) (end 94.01 75.51) (width 0.25) (layer "F.Cu") (net 16))
   (segment (start 94.01 75.51) (end 88.202501 69.702501) (width 0.25) (layer "F.Cu") (net 16))
+  (segment (start 62.6 67.4) (end 65.8 67.4) (width 0.25) (layer "F.Cu") (net 17))
   (segment (start 65.8 67.4) (end 66.602499 68.202499) (width 0.25) (layer "F.Cu") (net 17))
   (segment (start 66.602499 68.202499) (end 72.201377 68.202499) (width 0.25) (layer "F.Cu") (net 17))
-  (segment (start 58.1 67.4) (end 65.8 67.4) (width 0.25) (layer "F.Cu") (net 17))
+  (segment (start 62.5 67.5) (end 62.6 67.4) (width 0.25) (layer "F.Cu") (net 17))
   (segment (start 66.1975 69.2025) (end 72.201377 69.2025) (width 0.25) (layer "F.Cu") (net 18))
   (segment (start 65.3 70.1) (end 66.1975 69.2025) (width 0.25) (layer "F.Cu") (net 18))
@@
   (segment (start 92.5 69.25) (end 93.98 70.73) (width 0.25) (layer "B.Cu") (net 32))
   (segment (start 93.98 70.73) (end 93.98 89) (width 0.25) (layer "B.Cu") (net 32))
-  (segment (start 99.1 88.99) (end 99.1 72.35) (width 0.25) (layer "F.Cu") (net 33))
-  (segment (start 99.1 72.35) (end 91.05 64.3) (width 0.25) (layer "F.Cu") (net 33))
-  (segment (start 99.09 89) (end 99.1 88.99) (width 0.25) (layer "F.Cu") (net 33))
-  (segment (start 59.1 66.1) (end 58.1 66.1) (width 0.25) (layer "F.Cu") (net 33))
-  (segment (start 60.9 64.3) (end 59.1 66.1) (width 0.25) (layer "F.Cu") (net 33))
-  (segment (start 91.05 64.3) (end 60.9 64.3) (width 0.25) (layer "F.Cu") (net 33))
+  (segment (start 64.4 64.3) (end 62.5 66.2) (width 0.25) (layer "F.Cu") (net 33))
+  (segment (start 89.3 64.3) (end 64.4 64.3) (width 0.25) (layer "F.Cu") (net 33))
+  (segment (start 96 71) (end 89.3 64.3) (width 0.25) (layer "F.Cu") (net 33))
+  (segment (start 96 79.5) (end 96 71) (width 0.25) (layer "F.Cu") (net 33))
+  (segment (start 99.09 89) (end 99.09 82.59) (width 0.25) (layer "F.Cu") (net 33))
+  (segment (start 99.09 82.59) (end 96 79.5) (width 0.25) (layer "F.Cu") (net 33))
   (zone (net 2) (net_name "/GND") (layers F&B.Cu) (hatch edge 0.508)
     (connect_pads (clearance 0.508))
@@
         (xy 105 84.25)
         (xy 50 84.25)
-        (xy 50 50)
-        (xy 105 50)
+        (xy 50 63)
+        (xy 105 63)
       )
     )
